Commit message: fixed inertia issue

File: hexapod_drake/urdf/hexapod_description.urdf (robot description, URDF)
Before this commit: robot hexapod, 19 links, 18 joints
Links:
- link body: mass 1 -> 3.126
- link link1: mass 1 -> 0.121
- link link10: mass 1 -> 0.121
- link link11: mass 1 -> 0.43
- link link12: mass 1 -> 0.624
- link link13: mass 1 -> 0.121
- link link14: mass 1 -> 0.43
- link link15: mass 1 -> 0.624
- link link16: mass 1 -> 0.121
- link link17: mass 1 -> 0.43
- link link18: mass 1 -> 0.624
- link link2: mass 1 -> 0.43
- link link3: mass 1 -> 0.624
- link link4: mass 1 -> 0.121
- link link5: mass 1 -> 0.43
- link link6: mass 1 -> 0.624
- link link7: mass 1 -> 0.121
- link link8: mass 1 -> 0.43
- link link9: mass 1 -> 0.624
Joints:
- joint joint1: limit lower=-1.0471975511965976 upper=1.0471975511965976 effort=87 velocity=2.3925 -> lower=-3.14 upper=3.14 effort=87 velocity=2.3925
